Commit message: shorten xacro code

File: urdf/snake_stl.urdf (robot description, URDF)
Before this commit: robot test_robot, 21 links, 20 joints
Links:
- removed link base_link
- removed link link_001
- removed link link_002
- removed link link_003
- removed link link_004
- removed link link_005
- removed link link_006
- removed link link_007
- removed link link_008
- removed link link_009
- removed link link_010
- added link bracket_001, mass 0.0060293114415; collision mesh filename=package://fall_sim_001/mesh/adaptor.stl; visual mesh filename=package://fall_sim_001/mesh/adaptor.stl
- added link bracket_002, mass 0.0060293114415; collision mesh filename=package://fall_sim_001/mesh/adaptor.stl; visual mesh filename=package://fall_sim_001/mesh/adaptor.stl
- added link bracket_003, mass 0.0060293114415; collision mesh filename=package://fall_sim_001/mesh/adaptor.stl; visual mesh filename=package://fall_sim_001/mesh/adaptor.stl
- added link bracket_004, mass 0.0060293114415; collision mesh filename=package://fall_sim_001/mesh/adaptor.stl; visual mesh filename=package://fall_sim_001/mesh/adaptor.stl
- added link bracket_005, mass 0.0060293114415; collision mesh filename=package://fall_sim_001/mesh/adaptor.stl; visual mesh filename=package://fall_sim_001/mesh/adaptor.stl
- added link bracket_006, mass 0.0060293114415; collision mesh filename=package://fall_sim_001/mesh/adaptor.stl; visual mesh filename=package://fall_sim_001/mesh/adaptor.stl
- added link bracket_007, mass 0.0060293114415; collision mesh filename=package://fall_sim_001/mesh/adaptor.stl; visual mesh filename=package://fall_sim_001/mesh/adaptor.stl
- added link bracket_008, mass 0.0060293114415; collision mesh filename=package://fall_sim_001/mesh/adaptor.stl; visual mesh filename=package://fall_sim_001/mesh/adaptor.stl
- added link bracket_009, mass 0.0060293114415; collision mesh filename=package://fall_sim_001/mesh/adaptor.stl; visual mesh filename=package://fall_sim_001/mesh/adaptor.stl
- added link bracket_010, mass 0.0060293114415; collision mesh filename=package://fall_sim_001/mesh/adaptor.stl; visual mesh filename=package://fall_sim_001/mesh/adaptor.stl
- added link world
- link dynamixel_001: mass 0.005 -> 0.023967239474; geometry collision mesh filename=package://fall_sim_001/mesh/dynamixel.stl; visual mesh filename=package://fall_sim_001/mesh/dynamixel.stl
- link dynamixel_002: mass 0.005 -> 0.023967239474; geometry collision mesh filename=package://fall_sim_001/mesh/dynamixel.stl; visual mesh filename=package://fall_sim_001/mesh/dynamixel.stl
- link dynamixel_003: mass 0.005 -> 0.023967239474; geometry collision mesh filename=package://fall_sim_001/mesh/dynamixel.stl; visual mesh filename=package://fall_sim_001/mesh/dynamixel.stl
- link dynamixel_004: mass 0.005 -> 0.023967239474; geometry collision mesh filename=package://fall_sim_001/mesh/dynamixel.stl; visual mesh filename=package://fall_sim_001/mesh/dynamixel.stl
- link dynamixel_005: mass 0.005 -> 0.023967239474; geometry collision mesh filename=package://fall_sim_001/mesh/dynamixel.stl; visual mesh filename=package://fall_sim_001/mesh/dynamixel.stl
- link dynamixel_101: mass 0.005 -> 0.023967239474; geometry collision mesh filename=package://fall_sim_001/mesh/dynamixel.stl; visual mesh filename=package://fall_sim_001/mesh/dynamixel.stl
- link dynamixel_102: mass 0.005 -> 0.023967239474; geometry collision mesh filename=package://fall_sim_001/mesh/dynamixel.stl; visual mesh filename=package://fall_sim_001/mesh/dynamixel.stl
- link dynamixel_103: mass 0.005 -> 0.023967239474; geometry collision mesh filename=package://fall_sim_001/mesh/dynamixel.stl; visual mesh filename=package://fall_sim_001/mesh/dynamixel.stl
- link dynamixel_104: mass 0.005 -> 0.023967239474; geometry collision mesh filename=package://fall_sim_001/mesh/dynamixel.stl; visual mesh filename=package://fall_sim_001/mesh/dynamixel.stl
- link dynamixel_105: mass 0.005 -> 0.023967239474; geometry collision mesh filename=package://fall_sim_001/mesh/dynamixel.stl; visual mesh filename=package://fall_sim_001/mesh/dynamixel.stl
Joints:
- joint fixed_000: parent base_link -> world
- joint fixed_001: parent link_001 -> bracket_001
- joint fixed_002: parent link_002 -> bracket_002
- joint fixed_003: parent link_003 -> bracket_003
- joint fixed_004: parent link_004 -> bracket_004
- joint fixed_005: parent link_005 -> bracket_005
- joint fixed_006: parent link_006 -> bracket_006
- joint fixed_007: parent link_007 -> bracket_007
- joint fixed_008: parent link_008 -> bracket_008
- joint fixed_009: parent link_009 -> bracket_009
- joint joint_001: child link_001 -> bracket_001
- joint joint_002: child link_002 -> bracket_002
- joint joint_003: child link_003 -> bracket_003
- joint joint_004: child link_004 -> bracket_004
- joint joint_005: child link_005 -> bracket_005
- joint joint_006: child link_006 -> bracket_006
- joint joint_007: child link_007 -> bracket_007
- joint joint_008: child link_008 -> bracket_008
- joint joint_009: child link_009 -> bracket_009
- joint joint_010: child link_010 -> bracket_010

File: urdf/snake_stl.xacro (robot description, xacro)
@@ -1,29 +1,116 @@
 <robot name="test_robot" xmlns:xacro="http://ros.org/wiki/xacro">
-  <xacro:property name="dynamixel" value="package://snake/mesh/dynamixel.stl"/>
-  <xacro:property name="mass_d" value="0.005" />
+  <xacro:property name="dynamixel" value="package://fall_sim_001/mesh/dynamixel.stl"/>
+  <xacro:property name="mass_d" value="0.023967239474" />
   <xacro:property name="width_d" value="0.024" />
   <xacro:property name="depth_d" value="0.024" />
   <xacro:property name="height_d" value="0.036" />
-	<xacro:property name="ixx_d" value="0.00000078" />
-	<xacro:property name="iyy_d" value="0.00000078" />
-  <xacro:property name="izz_d" value="0.00000048" />
+	<xacro:property name="ixx_d" value="0.0000035392036062" />
+	<xacro:property name="iyy_d" value="0.0000032067700889" />
+  <xacro:property name="izz_d" value="0.0000025171567719" />
   <xacro:property name="gear" value="1" />
-  <xacro:property name="adaptor" value="package://snake/mesh/adaptor.stl"/>
-  <xacro:property name="mass_a" value="0.001" />
+  <xacro:property name="adaptor" value="package://fall_sim_001/mesh/adaptor.stl"/>
+  <xacro:property name="mass_a" value="0.0060293114415" />
   <xacro:property name="width_a" value="0.018" />
   <xacro:property name="depth_a" value="0.035" />
   <xacro:property name="height_a" value="0.015" />
-  <xacro:property name="ixx_a" value="0.000000120" />
-  <xacro:property name="iyy_a" value="0.000000046" />
-  <xacro:property name="izz_a" value="0.000000129" />
-	<link name="base_link"/>
-<xacro:macro name="dynamixel_link" params="suffix">
-      <link name="${suffix}">
+  <xacro:property name="ixx_a" value="0.0000014057440439" />
+  <xacro:property name="iyy_a" value="0.000001144769055" />
+  <xacro:property name="izz_a" value="0.0000005779531603" />
+  <xacro:property name="fixed_pos" value="0.046" />
+  <!-- 定義するdynamixelの名前 -->
+  <xacro:property name="dynamixel_names" value="${[
+                                        'dynamixel_001',
+                                        'dynamixel_101',
+                                        'dynamixel_002',
+                                        'dynamixel_102',
+                                        'dynamixel_003',
+                                        'dynamixel_103',
+                                        'dynamixel_004',
+                                        'dynamixel_104',
+                                        'dynamixel_005',
+                                        'dynamixel_105'
+                                          ]}" />
+  <!-- 定義するbracketの名前 -->
+  <xacro:property name="bracket_names" value="${[
+                                        'bracket_001',
+                                        'bracket_002',
+                                        'bracket_003',
+                                        'bracket_004',
+                                        'bracket_005',
+                                        'bracket_006',
+                                        'bracket_007',
+                                        'bracket_008',
+                                        'bracket_009',
+                                        'bracket_010'
+                                          ]}" />
+  <xacro:property name="joint_setting" value="${[
+                ['joint_001', 'dynamixel_001', 'bracket_001'],
+                ['fixed_001', 'bracket_001', 'dynamixel_101', 'odd'],
+                ['joint_002', 'dynamixel_101', 'bracket_002'],
+                ['fixed_002', 'bracket_002', 'dynamixel_002', 'even'],
+                ['joint_003', 'dynamixel_002', 'bracket_003'],
+                ['fixed_003', 'bracket_003', 'dynamixel_102', 'odd'],
+                ['joint_004', 'dynamixel_102', 'bracket_004'],
+                ['fixed_004', 'bracket_004', 'dynamixel_003', 'even'],
+                ['joint_005', 'dynamixel_003', 'bracket_005'],
+                ['fixed_005', 'bracket_005', 'dynamixel_103', 'odd'],
+                ['joint_006', 'dynamixel_103', 'bracket_006'],
+                ['fixed_006', 'bracket_006', 'dynamixel_004', 'even'],
+                ['joint_007', 'dynamixel_004', 'bracket_007'],
+                ['fixed_007', 'bracket_007', 'dynamixel_104', 'odd'],
+                ['joint_008', 'dynamixel_104', 'bracket_008'],
+                ['fixed_008', 'bracket_008', 'dynamixel_005', 'even'],
+                ['joint_009', 'dynamixel_005', 'bracket_009'],
+                ['fixed_009', 'bracket_009', 'dynamixel_105', 'odd'],
+                ['joint_010', 'dynamixel_105', 'bracket_010']
+                                              ]}" />
+	<link name="world"/>
+  <!-- マクロ関数の定義 -->
+  <!-- dynamixelの定義を作るマクロ関数 -->
+  <xacro:macro name="dynamixel_definition" params="items:=^">
+    <xacro:if value="${items}">
+      <!-- pop: listから取り出し -->
+      <xacro:property name="item" value="${items.pop(0)}"/>
+      <!-- link名 -->
+      <link name="${item}">
+        <!-- 見た目 -->
+        <visual>
+          <geometry>
+            <mesh filename = "${dynamixel}"/>
+          </geometry>
+          <material name="red">
+            <color rgba="0.7 0.0 0.0 1.0"/>
+          </material>
+                <origin rpy="0 0 0" xyz="0 0 0"/>
+        </visual>
+        <!--物理的特性-->
+        <!--干渉-->
+        <collision>
+          <geometry>
+            <mesh filename = "${dynamixel}"/>
+          </geometry>
+        </collision>
+        <!--慣性-->
+        <inertial>
+          <mass value="${mass_d}"/>
+          <inertia ixx="${ixx_d}" iyy="${iyy_d}" izz="${izz_d}" ixy="0" ixz="0" iyz="0"/>
+        </inertial>
+      </link>
+      <!-- 再帰 -->
+      <xacro:dynamixel_definition/>
+    </xacro:if>
+  </xacro:macro>
+  <!--Bracketの定義を作るマクロ関数-->
+  <xacro:macro name="bracket_definition" params="items:=^">
+    <xacro:if value="${items}">
+      <!-- pop: listから取り出し -->
+      <xacro:property name="item" value="${items.pop(0)}"/>
+      <link name="${item}">
       <visual>
         <geometry>
-          <mesh filename = "${dynamixel}"/>
+          <mesh filename = "${adaptor}"/>
         </geometry>
-        <material name="red">
-          <color rgba="0.7 0.0 0.0 1.0"/>
+        <material name="silver">
+          <color rgba="0.75 0.75 0.75 1"/>
         </material>
               <origin rpy="0 0 0" xyz="0 0 0"/>
@@ -33,366 +120,68 @@
       <collision>
         <geometry>
-          <mesh filename = "${dynamixel}"/>
+          <mesh filename = "${adaptor}"/>
         </geometry>
       </collision>
       <!--慣性-->
       <inertial>
-        <mass value="${mass_d}"/>
-        <inertia ixx="${ixx_d}" iyy="${iyy_d}" izz="${izz_d}" ixy="0" ixz="0" iyz="0"/>
+        <mass value="${mass_a}"/>
+        <inertia ixx="${ixx_a}" iyy="${iyy_a}" izz="${izz_a}" ixy="0" ixz="0" iyz="0"/>
       </inertial>
     </link>
-</xacro:macro>
-<!--Dynamixelの定義-->
-<!--リンク1~10-->
-<xacro:dynamixel_link suffix="dynamixel_001" />
-<xacro:dynamixel_link suffix="dynamixel_101" />
-<xacro:dynamixel_link suffix="dynamixel_002" />
-<xacro:dynamixel_link suffix="dynamixel_102" />
-<xacro:dynamixel_link suffix="dynamixel_003" />
-<xacro:dynamixel_link suffix="dynamixel_103" />
-<xacro:dynamixel_link suffix="dynamixel_004" />
-<xacro:dynamixel_link suffix="dynamixel_104" />
-<xacro:dynamixel_link suffix="dynamixel_005" />
-<xacro:dynamixel_link suffix="dynamixel_105" />
-<xacro:macro name="adaptor_link" params="suffix">
-    <link name="${suffix}">
-    <visual>
-      <geometry>
-        <mesh filename = "${adaptor}"/>
-      </geometry>
-      <material name="silver">
-        <color rgba="0.75 0.75 0.75 1"/>
-      </material>
-            <origin rpy="0 0 0" xyz="0 0 0"/>
-    </visual>
-    <!--物理的特性-->
-    <!--干渉-->
-    <collision>
-      <geometry>
-        <mesh filename = "${adaptor}"/>
-      </geometry>
-    </collision>
-    <!--慣性-->
-    <inertial>
-      <mass value="${mass_a}"/>
-      <inertia ixx="${ixx_a}" iyy="${iyy_a}" izz="${izz_a}" ixy="0" ixz="0" iyz="0"/>
-    </inertial>
-  </link>
-</xacro:macro>
-<!--アダプタの定義-->
-<!--リンク1-10 -->
-<xacro:dynamixel_link suffix="link_001" />
-<xacro:dynamixel_link suffix="link_002" />
-<xacro:dynamixel_link suffix="link_003" />
-<xacro:dynamixel_link suffix="link_004" />
-<xacro:dynamixel_link suffix="link_005" />
-<xacro:dynamixel_link suffix="link_006" />
-<xacro:dynamixel_link suffix="link_007" />
-<xacro:dynamixel_link suffix="link_008" />
-<xacro:dynamixel_link suffix="link_009" />
-<xacro:dynamixel_link suffix="link_010" />
-	<!--ジョイント設定-->
-	<!--ワールドとリンク1-->
-	<joint name="fixed_000" type="fixed">
-		<parent link="base_link"/>
-		<child  link="dynamixel_001"/>
-		<origin xyz="0 0 0" rpy="0 0 ${-pi/2}"/>
-    	<limit lower="${-pi/2}" upper="${pi/2}" effort="0" velocity="0"/>
-	</joint>
-	<!--Dynamixel1とリンク1-->
-	<joint name="joint_001" type="revolute">
-    <axis xyz="0 1 0"/>   <!--pitch-->
-		<parent link="dynamixel_001"/>
-		<child  link="link_001"/>
-		<origin xyz="0 0 0" rpy="0 0 0"/>
-    	<limit lower="${-pi/2}" upper="${pi/2}" effort="0" velocity="0"/>
-	</joint>
-  <!--リンク1とDynamixel101-->
-  <joint name="fixed_001" type="fixed">
-    <parent link="link_001"/>
-    <child  link="dynamixel_101"/>
-    <origin xyz="0.046 0 0" rpy="${pi/2} 0 0"/>
+    <!-- 再帰 -->
+    <xacro:bracket_definition/>
+    </xacro:if>
+  </xacro:macro>
+  <!-- ジョイントを定義するマクロ関数 -->
+  <xacro:macro name="joint_definition" params="items:=^">
+    <xacro:if value="${items}">
+      <!-- pop: listから取り出し -->
+      <xacro:property name="config" value="${items.pop(0)}"/>
+      <xacro:property name="name" value="${config[0]}"/>
+      <xacro:property name="parent" value="${config[1]}"/>
+      <xacro:property name="child" value="${config[2]}"/>
+      <xacro:if value="${'fixed' in name}">
+        <xacro:property name="flag" value="${config[3]}"/>
+        <xacro:property name="joint_type" value="fixed"/>
+        <xacro:property name="x" value="${fixed_pos}"/>
+        <xacro:if value="${flag == 'odd'}">
+          <xacro:property name="joint_type" value="fixed"/>
+          <xacro:property name="rpy" value="${pi/2} 0 0"/>
+        </xacro:if>
+        <xacro:if value="${flag == 'even'}">
+          <xacro:property name="joint_type" value="fixed"/>
+          <xacro:property name="rpy" value="${-pi/2} 0 0"/>
+        </xacro:if>
+      </xacro:if>
+      <xacro:if value="${'joint' in name}">
+        <xacro:property name="joint_type" value="revolute"/>
+        <xacro:property name="x" value="${0}"/>
+        <xacro:property name="rpy" value="0 0 0"/>
+      </xacro:if>
+      <joint name="${name}" type="${joint_type}">
+        <xacro:if value="${'joint' in name}">
+          <axis xyz="0 1 0"/>
+        </xacro:if>
+        <parent link="${parent}"/>
+        <child  link="${child}"/>
+        <origin xyz="${x} 0 0" rpy="${rpy}"/>
+          <limit lower="${-pi/2}" upper="${pi/2}" effort="0" velocity="0"/>
+      </joint>
+    <!-- 再帰 -->
+    <xacro:joint_definition/>
+    </xacro:if>
+  </xacro:macro>
+  <!--Dynamixelの定義-->
+  <xacro:dynamixel_definition items="${list(dynamixel_names)}"/>
+  <!--ブラケットの定義-->
+  <xacro:bracket_definition items="${list(bracket_names)}"/>
+  <!--ジョイントの定義-->
+  <!--ワールドとリンク1-->
+  <joint name="fixed_000" type="fixed">
+    <parent link="world"/>
+    <child  link="dynamixel_001"/>
+    <origin xyz="0 0 0" rpy="0 0 ${-pi/2}"/>
       <limit lower="${-pi/2}" upper="${pi/2}" effort="0" velocity="0"/>
   </joint>
-	<!--Dynamixel101とリンク2-->
-	<joint name="joint_002" type="revolute">
-    <axis xyz="0 1 0"/>   <!--yaw-->
-		<parent link="dynamixel_101"/>
-		<child  link="link_002"/>
-		<origin xyz="0 0 0" rpy="0 0 0"/>
-    	<limit lower="${-pi/2}" upper="${pi/2}" effort="0" velocity="0"/>
-	</joint>
-  <!--リンク2とDynamixel2-->
-  <joint name="fixed_002" type="fixed">
-    <parent link="link_002"/>
-    <child  link="dynamixel_002"/>
-    <origin xyz="0.046 0 0" rpy="${-pi/2} 0 0"/>
-      <limit lower="${-pi/2}" upper="${pi/2}" effort="0" velocity="0"/>
-  </joint>
-  <!--Dynamixel2とリンク3-->
-  <joint name="joint_003" type="revolute">
-    <axis xyz="0 1 0"/>   <!--pitch-->
-    <parent link="dynamixel_002"/>
-    <child  link="link_003"/>
-    <origin xyz="0 0 0" rpy="0 0 0"/>
-      <limit lower="${-pi/2}" upper="${pi/2}" effort="0" velocity="0"/>
-  </joint>
-  <!--リンク3とDynamixel102-->
-  <joint name="fixed_003" type="fixed">
-    <parent link="link_003"/>
-    <child  link="dynamixel_102"/>
-    <origin xyz="0.046 0 0" rpy="${pi/2} 0 0"/>
-      <limit lower="${-pi/2}" upper="${pi/2}" effort="0" velocity="0"/>
-  </joint>
-  <!--Dynamixel102とリンク4-->
-  <joint name="joint_004" type="revolute">
-    <axis xyz="0 1 0"/>   <!--yaw-->
-    <parent link="dynamixel_102"/>
-    <child  link="link_004"/>
-    <origin xyz="0 0 0" rpy="0 0 0"/>
-      <limit lower="${-pi/2}" upper="${pi/2}" effort="0" velocity="0"/>
-  </joint>
-  <!--リンク4とDynamixel3-->
-  <joint name="fixed_004" type="fixed">
-    <parent link="link_004"/>
-    <child  link="dynamixel_003"/>
-    <origin xyz="0.046 0 0" rpy="${-pi/2} 0 0"/>
-      <limit lower="${-pi/2}" upper="${pi/2}" effort="0" velocity="0"/>
-  </joint>
-  <!--Dynamixel3とリンク5-->
-  <joint name="joint_005" type="revolute">
-    <axis xyz="0 1 0"/>   <!--pitch-->
-    <parent link="dynamixel_003"/>
-    <child  link="link_005"/>
-    <origin xyz="0 0 0" rpy="0 0 0"/>
-      <limit lower="${-pi/2}" upper="${pi/2}" effort="0" velocity="0"/>
-  </joint>
-  <!--リンク5とDynamixel103-->
-  <joint name="fixed_005" type="fixed">
-    <parent link="link_005"/>
-    <child  link="dynamixel_103"/>
-    <origin xyz="0.046 0 0" rpy="${pi/2} 0 0"/>
-      <limit lower="${-pi/2}" upper="${pi/2}" effort="0" velocity="0"/>
-  </joint>
-  <!--Dynamixel103とリンク6-->
-  <joint name="joint_006" type="revolute">
-    <axis xyz="0 1 0"/>   <!--yaw-->
-    <parent link="dynamixel_103"/>
-    <child  link="link_006"/>
-    <origin xyz="0 0 0" rpy="0 0 0"/>
-      <limit lower="${-pi/2}" upper="${pi/2}" effort="0" velocity="0"/>
-  </joint>
-  <!--リンク6とDynamixel4-->
-  <joint name="fixed_006" type="fixed">
-    <parent link="link_006"/>
-    <child  link="dynamixel_004"/>
-    <origin xyz="0.046 0 0" rpy="${-pi/2} 0 0"/>
-      <limit lower="${-pi/2}" upper="${pi/2}" effort="0" velocity="0"/>
-  </joint>
-  <!--Dynamixel4とリンク7-->
-  <joint name="joint_007" type="revolute">
-    <axis xyz="0 1 0"/>   <!--pitch-->
-    <parent link="dynamixel_004"/>
-    <child  link="link_007"/>
-    <origin xyz="0 0 0" rpy="0 0 0"/>
-      <limit lower="${-pi/2}" upper="${pi/2}" effort="0" velocity="0"/>
-  </joint>
-  <!--リンク7とDynamixel104-->
-  <joint name="fixed_007" type="fixed">
-    <parent link="link_007"/>
-    <child  link="dynamixel_104"/>
-    <origin xyz="0.046 0 0" rpy="${pi/2} 0 0"/>
-      <limit lower="${-pi/2}" upper="${pi/2}" effort="0" velocity="0"/>
-  </joint>
-  <!--Dynamixel104とリンク8-->
-  <joint name="joint_008" type="revolute">
-    <axis xyz="0 1 0"/>   <!--yaw-->
-    <parent link="dynamixel_104"/>
-    <child  link="link_008"/>
-    <origin xyz="0 0 0" rpy="0 0 0"/>
-      <limit lower="${-pi/2}" upper="${pi/2}" effort="0" velocity="0"/>
-  </joint>
-  <!--リンク8とDynamixel5-->
-  <joint name="fixed_008" type="fixed">
-    <parent link="link_008"/>
-    <child  link="dynamixel_005"/>
-    <origin xyz="0.046 0 0" rpy="${-pi/2} 0 0"/>
-      <limit lower="${-pi/2}" upper="${pi/2}" effort="0" velocity="0"/>
-  </joint>
-  <!--Dynamixel5とリンク9-->
-  <joint name="joint_009" type="revolute">
-    <axis xyz="0 1 0"/>   <!--pitch-->
-    <parent link="dynamixel_005"/>
-    <child  link="link_009"/>
-    <origin xyz="0 0 0" rpy="0 0 0"/>
-      <limit lower="${-pi/2}" upper="${pi/2}" effort="0" velocity="0"/>
-  </joint>
-  <!--リンク9とDynamixel105-->
-  <joint name="fixed_009" type="fixed">
-    <parent link="link_009"/>
-    <child  link="dynamixel_105"/>
-    <origin xyz="0.046 0 0" rpy="${pi/2} 0 0"/>
-      <limit lower="${-pi/2}" upper="${pi/2}" effort="0" velocity="0"/>
-  </joint>
-  <!--Dynamixel105とリンク10-->
-  <joint name="joint_010" type="revolute">
-    <axis xyz="0 1 0"/>   <!--yaw-->
-    <parent link="dynamixel_105"/>
-    <child  link="link_010"/>
-    <origin xyz="0 0 0" rpy="0 0 0"/>
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