Commit message: shorten xacro code

File: urdf/snake_stl.urdf (robot description, URDF)
Before this commit: robot test_robot, 21 links, 20 joints
Links:
- link bracket_001: geometry collision mesh filename=package://snake/mesh/adaptor.stl; visual mesh filename=package://snake/mesh/adaptor.stl
- link bracket_002: geometry collision mesh filename=package://snake/mesh/adaptor.stl; visual mesh filename=package://snake/mesh/adaptor.stl
- link bracket_003: geometry collision mesh filename=package://snake/mesh/adaptor.stl; visual mesh filename=package://snake/mesh/adaptor.stl
- link bracket_004: geometry collision mesh filename=package://snake/mesh/adaptor.stl; visual mesh filename=package://snake/mesh/adaptor.stl
- link bracket_005: geometry collision mesh filename=package://snake/mesh/adaptor.stl; visual mesh filename=package://snake/mesh/adaptor.stl
- link bracket_006: geometry collision mesh filename=package://snake/mesh/adaptor.stl; visual mesh filename=package://snake/mesh/adaptor.stl
- link bracket_007: geometry collision mesh filename=package://snake/mesh/adaptor.stl; visual mesh filename=package://snake/mesh/adaptor.stl
- link bracket_008: geometry collision mesh filename=package://snake/mesh/adaptor.stl; visual mesh filename=package://snake/mesh/adaptor.stl
- link bracket_009: geometry collision mesh filename=package://snake/mesh/adaptor.stl; visual mesh filename=package://snake/mesh/adaptor.stl
- link bracket_010: geometry collision mesh filename=package://snake/mesh/adaptor.stl; visual mesh filename=package://snake/mesh/adaptor.stl
- link dynamixel_001: geometry collision mesh filename=package://snake/mesh/dynamixel.stl; visual mesh filename=package://snake/mesh/dynamixel.stl
- link dynamixel_002: geometry collision mesh filename=package://snake/mesh/dynamixel.stl; visual mesh filename=package://snake/mesh/dynamixel.stl
- link dynamixel_003: geometry collision mesh filename=package://snake/mesh/dynamixel.stl; visual mesh filename=package://snake/mesh/dynamixel.stl
- link dynamixel_004: geometry collision mesh filename=package://snake/mesh/dynamixel.stl; visual mesh filename=package://snake/mesh/dynamixel.stl
- link dynamixel_005: geometry collision mesh filename=package://snake/mesh/dynamixel.stl; visual mesh filename=package://snake/mesh/dynamixel.stl
- link dynamixel_101: geometry collision mesh filename=package://snake/mesh/dynamixel.stl; visual mesh filename=package://snake/mesh/dynamixel.stl
- link dynamixel_102: geometry collision mesh filename=package://snake/mesh/dynamixel.stl; visual mesh filename=package://snake/mesh/dynamixel.stl
- link dynamixel_103: geometry collision mesh filename=package://snake/mesh/dynamixel.stl; visual mesh filename=package://snake/mesh/dynamixel.stl
- link dynamixel_104: geometry collision mesh filename=package://snake/mesh/dynamixel.stl; visual mesh filename=package://snake/mesh/dynamixel.stl
- link dynamixel_105: geometry collision mesh filename=package://snake/mesh/dynamixel.stl; visual mesh filename=package://snake/mesh/dynamixel.stl

File: urdf/snake_stl.xacro (robot description, xacro)
@@ -1,4 +1,4 @@
 <robot name="test_robot" xmlns:xacro="http://ros.org/wiki/xacro">
-  <xacro:property name="dynamixel" value="package://fall_sim_001/mesh/dynamixel.stl"/>
+  <xacro:property name="dynamixel" value="package://snake/mesh/dynamixel.stl"/>
   <xacro:property name="mass_d" value="0.023967239474" />
   <xacro:property name="width_d" value="0.024" />
@@ -9,5 +9,5 @@
   <xacro:property name="izz_d" value="0.0000025171567719" />
   <xacro:property name="gear" value="1" />
-  <xacro:property name="adaptor" value="package://fall_sim_001/mesh/adaptor.stl"/>
+  <xacro:property name="adaptor" value="package://snake/mesh/adaptor.stl"/>
   <xacro:property name="mass_a" value="0.0060293114415" />
   <xacro:property name="width_a" value="0.018" />

Commit message: modified

File: urdf/snake_stl.urdf (robot description, URDF)
Before this commit: robot test_robot, 21 links, 20 joints
Links:
- link bracket_001: geometry collision mesh filename=package://Rviz_snake/mesh/adaptor.stl; visual mesh filename=package://Rviz_snake/mesh/adaptor.stl
- link bracket_002: geometry collision mesh filename=package://Rviz_snake/mesh/adaptor.stl; visual mesh filename=package://Rviz_snake/mesh/adaptor.stl
- link bracket_003: geometry collision mesh filename=package://Rviz_snake/mesh/adaptor.stl; visual mesh filename=package://Rviz_snake/mesh/adaptor.stl
- link bracket_004: geometry collision mesh filename=package://Rviz_snake/mesh/adaptor.stl; visual mesh filename=package://Rviz_snake/mesh/adaptor.stl
- link bracket_005: geometry collision mesh filename=package://Rviz_snake/mesh/adaptor.stl; visual mesh filename=package://Rviz_snake/mesh/adaptor.stl
- link bracket_006: geometry collision mesh filename=package://Rviz_snake/mesh/adaptor.stl; visual mesh filename=package://Rviz_snake/mesh/adaptor.stl
- link bracket_007: geometry collision mesh filename=package://Rviz_snake/mesh/adaptor.stl; visual mesh filename=package://Rviz_snake/mesh/adaptor.stl
- link bracket_008: geometry collision mesh filename=package://Rviz_snake/mesh/adaptor.stl; visual mesh filename=package://Rviz_snake/mesh/adaptor.stl
- link bracket_009: geometry collision mesh filename=package://Rviz_snake/mesh/adaptor.stl; visual mesh filename=package://Rviz_snake/mesh/adaptor.stl
- link bracket_010: geometry collision mesh filename=package://Rviz_snake/mesh/adaptor.stl; visual mesh filename=package://Rviz_snake/mesh/adaptor.stl
- link dynamixel_001: geometry collision mesh filename=package://Rviz_snake/mesh/dynamixel.stl; visual mesh filename=package://Rviz_snake/mesh/dynamixel.stl
- link dynamixel_002: geometry collision mesh filename=package://Rviz_snake/mesh/dynamixel.stl; visual mesh filename=package://Rviz_snake/mesh/dynamixel.stl
- link dynamixel_003: geometry collision mesh filename=package://Rviz_snake/mesh/dynamixel.stl; visual mesh filename=package://Rviz_snake/mesh/dynamixel.stl
- link dynamixel_004: geometry collision mesh filename=package://Rviz_snake/mesh/dynamixel.stl; visual mesh filename=package://Rviz_snake/mesh/dynamixel.stl
- link dynamixel_005: geometry collision mesh filename=package://Rviz_snake/mesh/dynamixel.stl; visual mesh filename=package://Rviz_snake/mesh/dynamixel.stl
- link dynamixel_101: geometry collision mesh filename=package://Rviz_snake/mesh/dynamixel.stl; visual mesh filename=package://Rviz_snake/mesh/dynamixel.stl
- link dynamixel_102: geometry collision mesh filename=package://Rviz_snake/mesh/dynamixel.stl; visual mesh filename=package://Rviz_snake/mesh/dynamixel.stl
- link dynamixel_103: geometry collision mesh filename=package://Rviz_snake/mesh/dynamixel.stl; visual mesh filename=package://Rviz_snake/mesh/dynamixel.stl
- link dynamixel_104: geometry collision mesh filename=package://Rviz_snake/mesh/dynamixel.stl; visual mesh filename=package://Rviz_snake/mesh/dynamixel.stl
- link dynamixel_105: geometry collision mesh filename=package://Rviz_snake/mesh/dynamixel.stl; visual mesh filename=package://Rviz_snake/mesh/dynamixel.stl
Joints:
- joint fixed_001: origin xyz=0.046 0 0 rpy=1.57079632679 0 0 -> xyz=0.021 0 0 rpy=1.57079632679 0 0
- joint fixed_002: origin xyz=0.046 0 0 rpy=-1.57079632679 0 0 -> xyz=0.021 0 0 rpy=-1.57079632679 0 0
- joint fixed_003: origin xyz=0.046 0 0 rpy=1.57079632679 0 0 -> xyz=0.021 0 0 rpy=1.57079632679 0 0
- joint fixed_004: origin xyz=0.046 0 0 rpy=-1.57079632679 0 0 -> xyz=0.021 0 0 rpy=-1.57079632679 0 0
- joint fixed_005: origin xyz=0.046 0 0 rpy=1.57079632679 0 0 -> xyz=0.021 0 0 rpy=1.57079632679 0 0
- joint fixed_006: origin xyz=0.046 0 0 rpy=-1.57079632679 0 0 -> xyz=0.021 0 0 rpy=-1.57079632679 0 0
- joint fixed_007: origin xyz=0.046 0 0 rpy=1.57079632679 0 0 -> xyz=0.021 0 0 rpy=1.57079632679 0 0
- joint fixed_008: origin xyz=0.046 0 0 rpy=-1.57079632679 0 0 -> xyz=0.021 0 0 rpy=-1.57079632679 0 0
- joint fixed_009: origin xyz=0.046 0 0 rpy=1.57079632679 0 0 -> xyz=0.021 0 0 rpy=1.57079632679 0 0
- joint joint_001: origin xyz=0 0 0 rpy=0 0 0 -> xyz=0.0248 0 0 rpy=0 0 0
- joint joint_002: origin xyz=0 0 0 rpy=0 0 0 -> xyz=0.0248 0 0 rpy=0 0 0
- joint joint_003: origin xyz=0 0 0 rpy=0 0 0 -> xyz=0.0248 0 0 rpy=0 0 0
- joint joint_004: origin xyz=0 0 0 rpy=0 0 0 -> xyz=0.0248 0 0 rpy=0 0 0
- joint joint_005: origin xyz=0 0 0 rpy=0 0 0 -> xyz=0.0248 0 0 rpy=0 0 0
- joint joint_006: origin xyz=0 0 0 rpy=0 0 0 -> xyz=0.0248 0 0 rpy=0 0 0
- joint joint_007: origin xyz=0 0 0 rpy=0 0 0 -> xyz=0.0248 0 0 rpy=0 0 0
- joint joint_008: origin xyz=0 0 0 rpy=0 0 0 -> xyz=0.0248 0 0 rpy=0 0 0
- joint joint_009: origin xyz=0 0 0 rpy=0 0 0 -> xyz=0.0248 0 0 rpy=0 0 0
- joint joint_010: origin xyz=0 0 0 rpy=0 0 0 -> xyz=0.0248 0 0 rpy=0 0 0

File: urdf/snake_stl.xacro (robot description, xacro)
@@ -1,4 +1,4 @@
 <robot name="test_robot" xmlns:xacro="http://ros.org/wiki/xacro">
-  <xacro:property name="dynamixel" value="package://snake/mesh/dynamixel.stl"/>
+  <xacro:property name="dynamixel" value="package://Rviz_snake/mesh/dynamixel.stl"/>
   <xacro:property name="mass_d" value="0.023967239474" />
 	<xacro:property name="ixx_d" value="3.5392036062e-06" />
@@ -9,13 +9,16 @@
   <xacro:property name="izx_d" value="0"/>
   <xacro:property name="gear" value="1" />
-  <xacro:property name="adaptor" value="package://snake/mesh/adaptor.stl"/>
+  <xacro:property name="adaptor" value="package://Rviz_snake/mesh/adaptor.stl"/>
   <xacro:property name="mass_a" value="0.0060293114415" />
   <xacro:property name="ixx_a" value="1.4057440439e-06" />
   <xacro:property name="iyy_a" value="1.144769055e-06" />
   <xacro:property name="izz_a" value="5.779531603e-07" />
-  <xacro:property name="ixx_a" value="0" />
-  <xacro:property name="iyy_a" value="0"/>
-  <xacro:property name="izz_a" value="0" />
-  <xacro:property name="fixed_pos" value="0.046" />
+  <xacro:property name="ixy_a" value="0" />
+  <xacro:property name="iyz_a" value="0"/>
+  <xacro:property name="izx_a" value="0" />
+  <!-- <xacro:property name="fixed_pos" value="0.0249" />
+  <xacro:property name="joint_pos" value="0.021" /> -->
+  <xacro:property name="fixed_pos" value="0.021" />
+  <xacro:property name="joint_pos" value="0.0248" />
   <!-- 定義するdynamixelの名前 -->
   <xacro:property name="dynamixel_names" value="${[
@@ -44,5 +47,5 @@
                                         'bracket_010'
                                           ]}" />
-  <xacro:property name="joint_setting" value="${[
+<xacro:property name="joint_setting" value="${[
                 ['joint_001', 'dynamixel_001', 'bracket_001'],
                 ['fixed_001', 'bracket_001', 'dynamixel_101', 'odd'],
@@ -182,5 +185,5 @@
       <xacro:if value="${'joint' in name}">
         <xacro:property name="joint_type" value="revolute"/>
-        <xacro:property name="x" value="${0}"/>
+        <xacro:property name="x" value="${joint_pos}"/>
         <xacro:property name="rpy" value="0 0 0"/>
       </xacro:if>
